File: SD65-PCB.kicad_pcb (KiCad board)
At the start: 2 copper layers, 24 parts, among them SW1 SW_Push, U1 ATmega32U4-AU, Y1 16MHz

Commit message: yes
Parts:
- moved C4 0.25 mm to (71.2, 55.5)
- moved C5 0.16 mm to (63.5, 55.5)
Routing:
- net GND: track 72.9 -> 143.2 mm
- net +5V: track 44.8 -> 101.7 mm, vias 2 -> 5
- net Net-(C5-Pad1): track 0.00 -> 12.3 mm
- net Net-(R3-Pad2): track 23.3 -> 34.6 mm
- net Net-(C4-Pad1): track 0.00 -> 8.95 mm
